File: pcb/mimic/adc_spi_esp12E.brd (EAGLE design)
At the start: 71.1 x 89.8 mm, 22 parts

Commit message: added .pdf .bpm of board and deleted garbage.
Parts:
- removed U1: (no value), esp8266modules:ESP12-SMD
Changed lines of the file:
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@@
 </element>
 <element name="X1" library="esp8266modules" package="ESP12-SMD" value="" x="36.83" y="16.51"/>
-<element name="U1" library="esp8266modules" package="ESP12-SMD" value="" x="-16.51" y="10.16"/>
 </elements>
 <signals>
