File: pcb/mimic/adc_spi_esp12E.sch (EAGLE design)
At the start: 22 parts

Commit message: added .pdf .bpm of board and deleted garbage.
Parts:
- removed U1: (no value), esp8266modules:ESP12SMD
Changed lines of the file:
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@@
 <part name="SUPPLY7" library="supply2" library_urn="urn:adsk.eagle:library:372" deviceset="VCC" device=""/>
 <part name="GND7" library="supply1" deviceset="GND" device=""/>
-<part name="U1" library="esp8266modules" deviceset="ESP12" device="SMD"/>
 </parts>
 <sheets>
@@
 </plain>
 <instances>
-<instance part="U1" gate="G$1" x="66.04" y="63.5"/>
 </instances>
 <busses>
